File: mcu_rev2.sch (EAGLE design)
At the start: 62 parts, among them CON1 1888687, IC1 CY8C4248LQI-BL583, J1 MINIPROG3, J2 SWD, J3 90131-0937, Y1 32.768KHz, Y2 24MHz

Commit message: ready for review and fab draft 1
Parts:
- RN1, RN2, RN3, RN4: value ACASA100021000P100 -> 4816P-T01-101LF; device ACASA100021000P100:ACASA100021000P100 -> 4816P-T01-101LF:4816P-T01-101LF
Connections:
- new net P0.0_O: J3.21, RN2.13
- new net P0.1_O: J3.22, RN2.14
- new net P0.2_O: J3.19, RN2.15
- new net P0.3_O: J3.20, RN2.16
- new net P0.4_O: J3.17, RN3.10
- new net P0.5_O: J3.18, RN3.11
- new net P1.0_O: J3.15, RN3.9
- new net P1.1_O: J3.16, RN3.12
- new net P1.2_O: J3.11, RN3.13
- new net P1.3_O: J3.12, RN3.14
- new net P1.6_O: J3.9, RN3.15
- new net P1.7_O: J3.10, RN3.16
- new net P2.0_O: J3.7, RN4.9
- new net P2.1_O: J3.8, RN4.10
- new net P2.2_O: J3.5, RN4.11
- new net P2.3_O: J3.6, RN4.12
- new net P2.4_O: J3.3, RN4.13
- new net P2.5_O: J3.4, RN4.14
- new net P2.6_O: J3.1, RN4.15
- new net P2.7_O: J3.2, RN4.16
- new net P3.0_O: J3.34, RN1.9
- new net P3.1_O: J3.33, RN1.10
- new net P3.2_O: J3.32, RN1.11
- new net P3.3_O: J3.31, RN1.12
- new net P3.4_O: J3.30, RN1.13
- new net P3.5_O: J3.29, RN1.14
- new net P3.6_O: J3.28, RN1.15
- new net P3.7_O: J3.27, RN1.16
- new net P4.0_O: J3.26, RN2.9
- new net P4.1_O: J3.25, RN2.10
- new net P5.0_O: J3.24, RN2.11
- new net P5.1_O: J3.23, RN2.12
- net P0.0: now also RN2.4; no longer J3.21, RN2.5
- net P0.1: now also RN2.3; no longer J3.22, RN2.6
- net P0.2: now also RN2.2; no longer J3.19, RN2.7
- net P0.3: now also RN2.1; no longer J3.20, RN2.8
- net P0.4: now also RN3.7; no longer J3.17, RN3.1
- net P0.5: now also RN3.6; no longer J3.18, RN3.2
- net P1.0: now also RN3.8; no longer J3.15, RN3.3
- net P1.1: now also RN3.5; no longer J3.16, RN3.4
- net P1.2: now also RN3.4; no longer J3.11, RN3.5
- net P1.3: now also RN3.3; no longer J3.12, RN3.6
- net P1.6: now also RN3.2; no longer J3.9, RN3.7
- net P1.7: now also RN3.1; no longer J3.10, RN3.8
- net P2.0: now also RN4.8; no longer J3.7, RN4.1
- net P2.1: now also RN4.7; no longer J3.8, RN4.2
- net P2.2: now also RN4.6; no longer J3.5, RN4.3
- net P2.3: now also RN4.5; no longer J3.6, RN4.4
- net P2.4: now also RN4.4; no longer J3.3, RN4.5
- net P2.5: now also RN4.3; no longer J3.4, RN4.6
- net P2.6: now also RN4.2; no longer J3.1, RN4.7
- net P2.7: now also RN4.1; no longer J3.2, RN4.8
- net P3.0: now also RN1.8; no longer J3.34, RN1.1
- net P3.1: now also RN1.7; no longer J3.33, RN1.2
- net P3.2: now also RN1.6; no longer J3.32, RN1.3
- net P3.3: now also RN1.5; no longer J3.31, RN1.4
- net P3.4: now also RN1.4; no longer J3.30, RN1.5
- net P3.5: now also RN1.3; no longer J3.29, RN1.6
- net P3.6: now also RN1.2; no longer J3.28, RN1.7
- net P3.7: now also RN1.1; no longer J3.27, RN1.8
- net P4.0: now also RN2.8; no longer J3.26, RN2.1
- net P4.1: now also RN2.7; no longer J3.25, RN2.2
- net P5.0: now also RN2.6; no longer J3.24, RN2.3
- net P5.1: now also RN2.5; no longer J3.23, RN2.4
Other:
- moved on the sheet: C21, C22, C26, C27, CON1, J1, J2
