File: mysch.brd (EAGLE design)
At the start: 212.1 x 89.8 mm, 155 parts, among them CON1 1888687, CON10 1888687, CON100 1888687, CON11 1888687, CON12 1888687, CON13 1888687, CON14 1888687, CON15 1888687, CON16 1888687, CON17 1888687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

Commit message: ready for review and fab draft 1
Routing:
- net V24: track 218.2 -> 741.9 mm, vias 1 -> 3
- net GND: track 1080.7 -> 1087.6 mm
- net Q11: track 60.0 -> 61.0 mm
